File: MMboard1.kicad_pcb (KiCad board)
At the start: 2 copper layers, 95.2 x 93.8 mm, 119 parts, among them J15 RESET, J16 AVR-ISP-6, J17 WS2812, J22 AREF, J25 TYPE-C-31-M-12, J33 RESET, J34 AVR-ISP-6, J35 WS2812, J4 AREF, J7 TYPE-C-31-M-12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

Commit message: Added CUI connector lib
Parts:
- added J18: SJ-43514-SMT, CUI:SJ-43514-SMT, F.Cu at (129.8, 21.6)
- added J36: SJ-43514-SMT, CUI:SJ-43514-SMT, F.Cu at (85.5, -52.5)
- J16, J34: value AVR-ISP-6 -> ISP
- moved SW2 240.0 mm to (237.9, -21.5)
- moved SW1 26.4 mm to (109.1, 28.9)
- moved BZ2 19.6 mm to (96.5, 19.1), turned to 180 degrees
- moved J16 15.2 mm to (79.7, 16.5), turned to 0 degrees
- moved BZ1 14.5 mm to (100.3, 19.1), turned to 180 degrees
- moved R14 14.4 mm to (124.8, 20.3)
- moved R13 14.4 mm to (124.8, 21.9)
- moved R1 13.8 mm to (119.9, 21.0)
- moved JP1 13.8 mm to (119.7, 17.6)
- moved JP2 13.8 mm to (122.3, 17.6)
- moved R2 13.8 mm to (122.1, 21.0)
- moved R12 11.4 mm to (103.6, 15.9)
- moved D2 9.79 mm to (122.4, 26.5), turned to 180 degrees
- moved J15 1.84 mm to (86.8, 19.3), turned to 180 degrees
- moved R5 1.40 mm to (84.2, 16.6)
Connections:
- J17 pad 2: (no net) -> /Left MCU/WS2812_out
- J25 pad A8: (no net) -> Net-(J25-PadA8)
- J25 pad B8: (no net) -> Net-(J25-PadB8)
- J35 pad 2: (no net) -> /Right MCU/WS2812_out
- J7 pad A8: (no net) -> Net-(J7-PadA8)
- J7 pad B8: (no net) -> Net-(J7-PadB8)
- SW1 pad A: (no net) -> /Left MCU/Enc_A
- SW1 pad B: (no net) -> /Left MCU/Enc_B
- SW1 pad MP: (no net) -> GND
- SW1 pad S1: (no net) -> /Left MCU/Enc_SW
- SW2 pad A: (no net) -> /Right MCU/Enc_A
- SW2 pad B: (no net) -> /Right MCU/Enc_B
- SW2 pad S1: (no net) -> /Right MCU/Enc_SW
- U1 pad 1: (no net) -> Net-(U1-Pad1)
- U1 pad 20: (no net) -> Net-(U1-Pad20)
- U1 pad 21: (no net) -> Net-(U1-Pad21)
- U1 pad 29: (no net) -> Net-(U1-Pad29)
- U1 pad 30: (no net) -> Net-(U1-Pad30)
- U1 pad 31: (no net) -> Net-(U1-Pad31)
- U1 pad 32: (no net) -> Net-(U1-Pad32)
- U1 pad 40: (no net) -> Net-(U1-Pad40)
- U1 pad 41: (no net) -> Net-(U1-Pad41)
- U1 pad 8: (no net) -> Net-(U1-Pad8)
- U2 pad 1: (no net) -> Net-(U2-Pad1)
- U2 pad 20: (no net) -> Net-(U2-Pad20)
- U2 pad 21: (no net) -> Net-(U2-Pad21)
- U2 pad 29: (no net) -> Net-(U2-Pad29)
- U2 pad 30: (no net) -> Net-(U2-Pad30)
- U2 pad 31: (no net) -> Net-(U2-Pad31)
- U2 pad 32: (no net) -> Net-(U2-Pad32)
- U2 pad 40: (no net) -> Net-(U2-Pad40)
- U2 pad 41: (no net) -> Net-(U2-Pad41)
- U2 pad 8: (no net) -> Net-(U2-Pad8)
Routing:
- net +5V: track 122.4 -> 166.9 mm, vias 10 -> 14
- net /Left MCU/~reset: track 44.8 -> 31.0 mm
- net /Left MCU/Rr_2: track 4.69 -> 17.1 mm, vias 0 -> 2
- net /Left MCU/Rr_1: track 1.56 -> 13.7 mm
- net /Left MCU/SDA: track 52.1 -> 59.6 mm
- net /Left MCU/SCK: track 37.9 -> 30.5 mm
- net /Left MCU/SCL: track 53.2 -> 58.1 mm
- net /Left MCU/MISO: track 35.0 -> 30.8 mm
- net /Left MCU/MOSI: track 40.1 -> 36.2 mm
- net /Left MCU/buzz: track 5.61 -> 2.49 mm
- net GND: track 56.3 -> 53.3 mm, vias 74 -> 63
- net Net-(D9-Pad1): track 43.6 -> 43.0 mm
- net Net-(D14-Pad1): track 97.7 -> 97.2 mm
