File: mystic_split40.kicad_pcb (KiCad board)
At the start: 2 copper layers, 220.5 x 98.8 mm, 207 parts, among them J15 RESET, J16 ISP, J17 WS2812, J18 SJ-43514-SMT, J22 AREF, J25 TYPE-C-31-M-12, J33 RESET, J34 ISP, J35 WS2812, J36 SJ-43514-SMT, J4 AREF, J7 TYPE-C-31-M-12, SW1 EC11E, SW2 EC11E, SW3 Reset, SW4 Reset, U1 ATmega32U4-AU, U2 ATmega32U4-AU, Y1 CSTNE16M0VH3L000R0, Y2 CSTNE16M0VH3L000R0

Commit message: Finished right-side, added BOM
Parts:
- removed the BZ3 at (-156.3, 100.3)
- removed the BZ4 at (-156.3, 96.5)
- removed the C4 at (-87.2, 121.5)
- removed the C5 at (180.2, 23.1)
- removed the C5 at (-109.6, 145.5)
- removed the C6 at (180.2, 21.6)
- removed the C6 at (-101.6, 131.2)
- removed the D15 at (-150.1, 130.2)
- removed the D16 at (-156.5, 130.2)
- removed the D17 at (-163.0, 130.2)
- removed the D18 at (-150.8, 139.2)
- removed the D19 at (-143.6, 130.2)
- removed the D20 at (-163.0, 134.8)
- removed the D21 at (-156.5, 134.8)
- removed the D22 at (-150.1, 134.8)
- removed the D23 at (-163.0, 139.3)
- removed the D24 at (-156.5, 139.3)
- removed the D26 at (-100.0, 145.3)
- removed the D28 at (-126.0, 121.8)
- removed the D3 at (-105.6, 136.1)
- removed the D4 at (246.4, 26.2)
- removed the D4 at (-91.9, 122.5)
- removed the F2 at (-131.3, 146.9)
- removed the J22 at (-131.7, 120.7)
- removed the J25 at (-114.0, 139.6)
- removed the J33 at (-96.8, 122.5)
- removed the J34 at (-115.8, 146.8)
- removed the J36 at (254.2, 21.6)
- removed the J36 at (-105.5, 91.8)
- removed J4: AREF, TestPoint:TestPoint_Pad_D1.0mm
- removed the MX21 at (-88.3, 161.2)
- removed the MX22 at (-107.4, 161.2)
- removed the MX23 at (-126.5, 161.2)
- removed the MX24 at (-145.5, 161.2)
- removed the MX25 at (-164.6, 161.2)
- removed the MX26 at (-88.3, 180.3)
- removed the MX27 at (-107.4, 180.3)
- removed the MX28 at (-126.5, 180.3)
- removed the MX29 at (-145.5, 180.3)
- removed the MX30 at (-164.6, 180.3)
- removed the MX31 at (-88.3, 199.3)
- removed the MX32 at (-107.4, 199.3)
- removed the MX33 at (-126.5, 199.3)
- removed the MX34 at (-145.5, 199.3)
- removed the MX35 at (-164.6, 199.3)
- removed the MX36 at (-88.3, 218.4)
- removed the MX37 at (-107.4, 218.4)
- removed the MX38 at (-126.5, 218.4)
- removed the MX39 at (-145.5, 218.4)
- removed the MX40 at (-164.6, 218.4)
- removed the MX42 at (-155.0, 218.4)
- removed the R15 at (-100.8, 133.7)
- removed the R16 at (179.3, 18.9)
- removed the R16 at (-106.0, 142.1)
- removed the R17 at (179.3, 15.5)
- removed the R17 at (-106.0, 139.6)
- removed the R18 at (-100.8, 136.2)
- removed the R19 at (180.1, 26.9)
- removed the R19 at (-92.0, 128.5)
- removed the R20 at (180.1, 28.5)
- removed the R20 at (-109.6, 148.0)
- removed the R21 at (-100.8, 138.7)
- removed the R22 at (-126.2, 146.5)
- removed the R23 at (248.9, 21.0)
- removed the R23 at (-96.5, 133.4)
- removed the R24 at (246.1, 23.6)
- removed the R24 at (-92.3, 126.0)
- removed the R4 at (-136.8, 135.1)
- removed the REF** at (134.0, 14.7)
- removed the REF** at (167.0, 14.7)
- removed the SW2 at (-73.3, 103.0)
- removed the SW4 at (-86.8, 141.4)
- removed the U2 at (-127.0, 138.0)
- removed the Y2 at (-96.6, 129.8)
- added C5: 100nF, Capacitor_SMD:C_0603_1608Metric_Pad1.05x0.95mm_HandSolder, F.Cu at (180.2, 26.4)
- added C6: 1uF, Capacitor_SMD:C_0603_1608Metric_Pad1.05x0.95mm_HandSolder, F.Cu at (180.2, 27.9)
- added D4: PRTR5V0U2X, Package_TO_SOT_SMD:SOT-143, F.Cu at (177.3, 22.9)
- added J1: RX, TestPoint:TestPoint_Pad_D1.0mm, B.Cu at (67.0, 19.5)
- added J2: TX, TestPoint:TestPoint_Pad_D1.0mm, B.Cu at (65.0, 19.5)
- added J3: RX, TestPoint:TestPoint_Pad_D1.0mm, B.Cu at (192.3, 19.5)
- added J36: SJ-43514-SMT, CUI:SJ-43514-SMT, F.Cu at (172.0, 21.6)
- added J5: TX, TestPoint:TestPoint_Pad_D1.0mm, B.Cu at (190.2, 19.5)
- added MX43: MX-NoLED, Ai03-MX:MXOnly-2U-Hotswap, F.Cu at (59.3, 102.0)
- added MX44: MX-NoLED, Ai03-MX:MXOnly-2U-Hotswap, F.Cu at (184.6, 102.0)
- added R16: 5k1, Resistor_SMD:R_0603_1608Metric_Pad1.05x0.95mm_HandSolder, F.Cu at (247.0, 15.5)
- added R17: 5k1, Resistor_SMD:R_0603_1608Metric_Pad1.05x0.95mm_HandSolder, F.Cu at (247.0, 18.9)
- added R19: 22R, Resistor_SMD:R_0603_1608Metric_Pad1.05x0.95mm_HandSolder, F.Cu at (192.2, 33.0)
- added R20: 22R, Resistor_SMD:R_0603_1608Metric_Pad1.05x0.95mm_HandSolder, F.Cu at (192.2, 31.4)
- added R23: 220R, Resistor_SMD:R_0603_1608Metric_Pad1.05x0.95mm_HandSolder, F.Cu at (177.7, 27.3)
- added R24: 220R, Resistor_SMD:R_0603_1608Metric_Pad1.05x0.95mm_HandSolder, F.Cu at (176.2, 27.3)
- J35: moved to B.Cu
- moved J35 298.9 mm to (178.0, 16.4), turned to 270 degrees
- moved F2 86.9 mm to (256.5, 25.5)
- moved D3 80.0 mm to (253.2, 24.3)
- moved J25 80.0 mm to (253.2, 16.3)
- renumbered J4 to J22, R5 to R15
Connections:
- BZ3 pad 1: Net-(BZ1-Pad1) -> Net-(BZ3-Pad1)
- BZ4 pad 1: /Left MCU/buzz -> /Right MCU/buzz
- C4 pad 2: Net-(C1-Pad2) -> Net-(C4-Pad2)
- D15 pad 1: Net-(D5-Pad1) -> Net-(D15-Pad1)
- D15 pad 2: Net-(D5-Pad2) -> Net-(D15-Pad2)
- D15 pad 3: /Left MCU/col4 -> /Matrix right/col4
- D16 pad 1: Net-(D6-Pad1) -> Net-(D16-Pad1)
- D16 pad 2: Net-(D6-Pad2) -> Net-(D16-Pad2)
- D16 pad 3: /Left MCU/col4 -> /Matrix right/col4
- D17 pad 1: Net-(D7-Pad1) -> Net-(D17-Pad1)
- D17 pad 2: Net-(D7-Pad2) -> Net-(D17-Pad2)
- D17 pad 3: /Left MCU/col3 -> /Matrix right/col3
- D18 pad 1: Net-(D8-Pad1) -> Net-(D18-Pad1)
- D18 pad 2: Net-(D8-Pad2) -> Net-(D18-Pad2)
- D18 pad 3: /Left MCU/col3 -> /Matrix right/col3
- D19 pad 1: Net-(D9-Pad1) -> Net-(D19-Pad1)
- D19 pad 2: Net-(D9-Pad2) -> Net-(D19-Pad2)
- D19 pad 3: /Left MCU/col2 -> /Matrix right/col2
- D20 pad 1: Net-(D10-Pad1) -> Net-(D20-Pad1)
- D20 pad 2: Net-(D10-Pad2) -> Net-(D20-Pad2)
- D20 pad 3: /Left MCU/col2 -> /Matrix right/col2
- D21 pad 1: Net-(D11-Pad1) -> Net-(D21-Pad1)
- D21 pad 2: Net-(D11-Pad2) -> Net-(D21-Pad2)
- D21 pad 3: /Left MCU/col1 -> /Matrix right/col1
- D22 pad 1: Net-(D12-Pad1) -> Net-(D22-Pad1)
- D22 pad 2: Net-(D12-Pad2) -> Net-(D22-Pad2)
- D22 pad 3: /Left MCU/col1 -> /Matrix right/col1
- D23 pad 1: Net-(D13-Pad1) -> Net-(D23-Pad1)
- D23 pad 2: Net-(D13-Pad2) -> Net-(D23-Pad2)
- D23 pad 3: /Left MCU/col0 -> /Matrix right/col0
- D24 pad 1: Net-(D14-Pad1) -> Net-(D24-Pad1)
- D24 pad 2: Net-(D14-Pad2) -> Net-(D24-Pad2)
- D24 pad 3: /Left MCU/col0 -> /Matrix right/col0
- D26 pad 1: Net-(D25-Pad1) -> Net-(D26-Pad1)
- D26 pad 2: /Left MCU/row0 -> /Matrix right/row0
- D28 pad 2: Net-(D27-Pad2) -> Net-(D28-Pad2)
- D3 pad 2: /Left MCU/Dd- -> /Right MCU/Dd-
- D3 pad 3: /Left MCU/Dd+ -> /Right MCU/Dd+
- J22 pad 1: Net-(J4-Pad1) -> (no net)
- J25 pad A5: Net-(J7-PadA5) -> Net-(J25-PadA5)
- J25 pad A6: /Left MCU/Dd+ -> /Right MCU/Dd+
- J25 pad A7: /Left MCU/Dd- -> /Right MCU/Dd-
- J25 pad B5: Net-(J7-PadB5) -> Net-(J25-PadB5)
- J25 pad B6: /Left MCU/Dd+ -> /Right MCU/Dd+
- J25 pad B7: /Left MCU/Dd- -> /Right MCU/Dd-
- J33 pad 2: /Left MCU/~reset -> /Right MCU/~reset
- J34 pad 1: /Left MCU/MISO -> /Right MCU/MISO
- J34 pad 3: /Left MCU/SCK -> /Right MCU/SCK
- J34 pad 4: /Left MCU/MOSI -> /Right MCU/MOSI
- J34 pad 5: /Left MCU/~reset -> /Right MCU/~reset
- MX21 pad 1: Net-(D13-Pad2) -> Net-(D23-Pad2)
- MX21 pad 2: /Left MCU/row0 -> /Matrix right/row0
- MX22 pad 1: Net-(D11-Pad2) -> Net-(D21-Pad2)
- MX22 pad 2: /Left MCU/row0 -> /Matrix right/row0
- MX23 pad 1: Net-(D9-Pad2) -> Net-(D19-Pad2)
- MX23 pad 2: /Left MCU/row0 -> /Matrix right/row0
- MX24 pad 1: Net-(D7-Pad2) -> Net-(D17-Pad2)
- MX24 pad 2: /Left MCU/row0 -> /Matrix right/row0
- MX25 pad 1: Net-(D5-Pad2) -> Net-(D15-Pad2)
- MX25 pad 2: /Left MCU/row0 -> /Matrix right/row0
- MX26 pad 1: Net-(D13-Pad1) -> Net-(D23-Pad1)
- MX26 pad 2: /Left MCU/row1 -> /Matrix right/row1
- MX27 pad 1: Net-(D11-Pad1) -> Net-(D21-Pad1)
- MX27 pad 2: /Left MCU/row1 -> /Matrix right/row1
- MX28 pad 1: Net-(D9-Pad1) -> Net-(D19-Pad1)
- MX28 pad 2: /Left MCU/row1 -> /Matrix right/row1
- MX29 pad 1: Net-(D7-Pad1) -> Net-(D17-Pad1)
- MX29 pad 2: /Left MCU/row1 -> /Matrix right/row1
- MX30 pad 1: Net-(D5-Pad1) -> Net-(D15-Pad1)
- MX30 pad 2: /Left MCU/row1 -> /Matrix right/row1
- MX31 pad 1: Net-(D14-Pad2) -> Net-(D24-Pad2)
- MX31 pad 2: /Left MCU/row2 -> /Matrix right/row2
- MX32 pad 1: Net-(D12-Pad2) -> Net-(D22-Pad2)
- MX32 pad 2: /Left MCU/row2 -> /Matrix right/row2
- MX33 pad 1: Net-(D10-Pad2) -> Net-(D20-Pad2)
- MX33 pad 2: /Left MCU/row2 -> /Matrix right/row2
- MX34 pad 1: Net-(D8-Pad2) -> Net-(D18-Pad2)
- MX34 pad 2: /Left MCU/row2 -> /Matrix right/row2
- MX35 pad 1: Net-(D6-Pad2) -> Net-(D16-Pad2)
- MX35 pad 2: /Left MCU/row2 -> /Matrix right/row2
- MX36 pad 1: Net-(D14-Pad1) -> Net-(D24-Pad1)
- MX36 pad 2: /Left MCU/row3 -> /Matrix right/row3
- MX37 pad 1: Net-(D12-Pad1) -> Net-(D22-Pad1)
- MX37 pad 2: /Left MCU/row3 -> /Matrix right/row3
- MX38 pad 1: Net-(D10-Pad1) -> Net-(D20-Pad1)
- MX38 pad 2: /Left MCU/row3 -> /Matrix right/row3
- MX39 pad 1: Net-(D8-Pad1) -> Net-(D18-Pad1)
- MX39 pad 2: /Left MCU/row3 -> /Matrix right/row3
- MX40 pad 1: Net-(D6-Pad1) -> Net-(D16-Pad1)
- MX40 pad 2: /Left MCU/row3 -> /Matrix right/row3
- MX42 pad 1: Net-(D6-Pad1) -> Net-(D16-Pad1)
- MX42 pad 2: /Left MCU/row3 -> /Matrix right/row3
- R15 pad 2: /Left MCU/~reset -> /Right MCU/~reset
- R18 pad 1: Net-(R8-Pad1) -> Net-(R18-Pad1)
- R18 pad 2: +5V -> GND
- R21 pad 2: Net-(R11-Pad2) -> Net-(R21-Pad2)
- R22 pad 1: Net-(BZ1-Pad1) -> Net-(BZ3-Pad1)
- R22 pad 2: /Left MCU/buzz -> /Right MCU/buzz
- R4 pad 1: Net-(D27-Pad2) -> Net-(D28-Pad2)
- R4 pad 2: /Left MCU/DFU_LED -> /Right MCU/DFU_LED
- SW2 pad A: /Left MCU/Enc_A -> /Right MCU/Enc_A
- SW2 pad B: /Left MCU/Enc_B -> /Right MCU/Enc_B
- SW2 pad S1: Net-(D25-Pad1) -> Net-(D26-Pad1)
- SW2 pad S2: /Left MCU/Enc_S1 -> /Right MCU/Enc_S1
- SW4 pad 1: /Left MCU/~reset -> /Right MCU/~reset
- U1 pad 16: Net-(U1-Pad16) -> /Left MCU/x+
- U1 pad 17: Net-(U1-Pad17) -> /Left MCU/x-
- U1 pad 20: (no net) -> Net-(J1-Pad1)
- U1 pad 21: (no net) -> Net-(J2-Pad1)
- U1 pad 42: Net-(J4-Pad1) -> (no net)
- U2 pad 1: /Left MCU/Enc_B -> /Right MCU/Enc_B
- U2 pad 10: /Left MCU/MOSI -> /Right MCU/MOSI
- U2 pad 11: /Left MCU/MISO -> /Right MCU/MISO
- U2 pad 12: Net-(R8-Pad1) -> Net-(R18-Pad1)
- U2 pad 13: /Left MCU/~reset -> /Right MCU/~reset
- U2 pad 16: Net-(U1-Pad16) -> /Right MCU/x+
- U2 pad 17: Net-(U1-Pad17) -> /Right MCU/x-
- U2 pad 18: /Left MCU/SCL -> /Right MCU/SCL
- U2 pad 19: /Left MCU/SDA -> /Right MCU/SDA
- U2 pad 20: (no net) -> Net-(J3-Pad1)
- U2 pad 21: (no net) -> Net-(J5-Pad1)
- U2 pad 22: /Left MCU/col0 -> /Matrix right/col0
- U2 pad 25: /Left MCU/col1 -> /Matrix right/col1
- U2 pad 26: /Left MCU/col2 -> /Matrix right/col2
- U2 pad 27: /Left MCU/col3 -> /Matrix right/col3
- U2 pad 28: /Left MCU/col4 -> /Matrix right/col4
- U2 pad 29: /Left MCU/DFU_LED -> /Right MCU/DFU_LED
- U2 pad 3: /Left MCU/D- -> /Right MCU/D-
- U2 pad 30: /Left MCU/WS2812_out -> /Right MCU/WS2812_out
- U2 pad 31: /Left MCU/buzz -> /Right MCU/buzz
- U2 pad 32: /Left MCU/Enc_S1 -> /Right MCU/Enc_S1
- U2 pad 33: Net-(R11-Pad2) -> Net-(R21-Pad2)
- U2 pad 36: /Left MCU/row0 -> /Matrix right/row0
- U2 pad 37: /Left MCU/row1 -> /Matrix right/row1
- U2 pad 38: /Left MCU/row2 -> /Matrix right/row2
- U2 pad 39: /Left MCU/row3 -> /Matrix right/row3
- U2 pad 4: /Left MCU/D+ -> /Right MCU/D+
- U2 pad 42: Net-(J4-Pad1) -> (no net)
- U2 pad 6: Net-(C1-Pad2) -> Net-(C4-Pad2)
- U2 pad 8: /Left MCU/Enc_A -> /Right MCU/Enc_A
- U2 pad 9: /Left MCU/SCK -> /Right MCU/SCK
- Y1 pad 1: Net-(U1-Pad17) -> /Left MCU/x-
- Y1 pad 3: Net-(U1-Pad16) -> /Left MCU/x+
- Y2 pad 1: Net-(U1-Pad17) -> /Right MCU/x-
- Y2 pad 3: Net-(U1-Pad16) -> /Right MCU/x+
Routing:
- net /Left MCU/row3: track 359.6 -> 194.4 mm, vias 6 -> 3
- net /Left MCU/row2: track 296.2 -> 148.1 mm, vias 6 -> 3
- net /Left MCU/row1: track 266.7 -> 133.4 mm, vias 6 -> 3
- net /Left MCU/row0: track 236.5 -> 118.2 mm, vias 4 -> 2
- net Net-(D24-Pad1): track 0.00 -> 114.2 mm, vias 0 -> 1
- net Net-(D6-Pad1): track 210.0 -> 105.0 mm, vias 2 -> 1
- net /Matrix right/row3: track 101.3 -> 193.6 mm, vias 0 -> 3
- net Net-(D12-Pad1): track 183.1 -> 91.6 mm, vias 2 -> 1
- net Net-(D22-Pad1): track 0.00 -> 91.6 mm, vias 0 -> 1
- net Net-(D16-Pad1): track 15.0 -> 105.0 mm, vias 0 -> 1
- net /Right MCU/Dd-: track 0.00 -> 85.2 mm, vias 0 -> 4
- net /Right MCU/Dd+: track 0.00 -> 84.5 mm, vias 0 -> 4
- net Net-(D14-Pad1): track 197.9 -> 114.3 mm, vias 2 -> 1
- net Net-(D24-Pad2): track 0.00 -> 81.7 mm, vias 0 -> 1
- net Net-(D14-Pad2): track 163.5 -> 81.7 mm, vias 2 -> 1
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Other:
- board text added: "V0.1"
- board text removed: "V1.0"
