File: MCU.sch (KiCad schematic (older format))
At the start: 34 parts, among them J1 RX, J15 RESET, J16 ISP, J17 WS2812, J18 SJ-43514-SMT, J2 TX, J7 TYPE-C-31-M-12, SW1 EC11E, SW3 Reset, U1 ATmega32U4-AU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

Commit message: regenerated gerbers
Parts:
- gave numbers to parts that had none: 2

Commit message: Started work on adding extra col
Parts:
- removed J4: F0, TestPoint:TestPoint_Pad_D1.0mm, symbol Connector_Generic:Conn_01x01
- added TP4: SCK, TestPoint:TestPoint_Pad_D1.0mm, symbol Connector:TestPoint
- added TP5: MOSI, TestPoint:TestPoint_Pad_D1.0mm, symbol Connector:TestPoint
- added TP6: MISO, TestPoint:TestPoint_Pad_D1.0mm, symbol Connector:TestPoint
- renumbered D1 to D29, D2 to D30, D25 to D31, D27 to D32
Connections:
- net DFU_LED: now also U1.41 (PF0); no longer U1.29 (PB5)
- net MISO: now also TP6.1
- net MOSI: now also TP5.1
- net SCK: now also TP4.1
- new net col5: U1.29 (PB5)
